File: lumiled_driver.brd (EAGLE design)
At the start: 55 x 38 mm, 17 parts, among them Q1 IRF520, Q2 2N3904, Q3 IRF520, Q4 2N3904, Q5 IRF520, Q6 2N3904

Commit message: -wow it's been a while since the last commit
Parts:
- R1, R2, R3, R4, R5, R6: device rcl:0204/7 -> resistor:0411/12
- moved Q2 12.3 mm to (26.8, 20.8)
- moved Q1 12.0 mm to (19.2, 22.8)
- moved Q3 11.9 mm to (19.2, 31.0)
- moved Q6 11.9 mm to (27.1, 11.2)
- moved Q4 11.9 mm to (27.1, 30.3)
- moved Q5 11.8 mm to (19.5, 14.5)
- moved R1 8.10 mm to (39.0, 17.8)
- moved R6 8.06 mm to (39.0, 13.0)
- moved R2 8.02 mm to (39.0, 22.5)
- moved R5 7.95 mm to (39.0, 8.25)
- moved R4 7.85 mm to (39.2, 32.0)
- moved R3 7.75 mm to (39.2, 27.2)
- moved C2 4.61 mm to (17.5, 35.0), turned to 0 degrees
- moved C1 4.42 mm to (11.8, 35.0), turned to 0 degrees
Routing:
- net N$10: track 27.5 -> 14.9 mm
- net N$27: track 25.3 -> 13.4 mm
- net N$26: track 30.2 -> 19.0 mm
- net GRN_PWM: track 52.9 -> 42.2 mm
- net RED_PWM: track 60.8 -> 53.0 mm
- net BLU_PWM: track 40.2 -> 34.0 mm
- net +VIN: track 33.1 -> 38.9 mm
- net N$21: track 13.4 -> 18.6 mm
- net N$17: track 28.7 -> 33.4 mm
- net N$18: track 30.5 -> 34.9 mm
- net N$19: track 28.6 -> 33.0 mm
- net N$20: track 13.8 -> 17.5 mm
- added copper zone on layer 16, net GND
Other:
- board size 55 x 38 mm -> 52.5 x 38 mm
- board text added: "Lumiled Driver V3.2"
- board text removed: "Lumiled Driver V3.1"

Commit message: -sent out to elecrow for fabrication
Parts:
- added C3: 100nF, rcl:C025-024X044
- added C4: 1uF, resistor:TT2D5
- added C5: 10uF, resistor:TT2D5
- added CN2: (no value), adafruit:DCJACK_2MM_PTH
- added D1: 1N4004, diode:DO41-10
- added IC1: (no value), v-reg:317TL
- added JP2: (no value), pinhead:1X03
- added Q10, Q11, Q12: 2N3904, transistor-npn:TO92
- added Q7, Q8, Q9: IRF520, transistor-power:TO220BV
- added R10, R11, R12, R13, R14, R7, R8, R9: (no value), resistor:0411/12
- added U$2: LUMILED_PARALLEL, lumiled_led:LED_PAR
- moved C1 0.50 mm to (11.8, 35.5)
- moved C2 0.50 mm to (17.5, 35.5)
- moved CN1 0.50 mm to (-3.00, 27.5)
- moved JP1 0.50 mm to (11.0, 3.50)
- moved Q1 0.50 mm to (19.2, 23.2)
- moved Q2 0.50 mm to (26.8, 21.2)
- moved Q3 0.50 mm to (19.2, 31.5)
- moved Q4 0.50 mm to (27.1, 30.8)
- moved Q5 0.50 mm to (19.5, 15.0)
- moved Q6 0.50 mm to (27.1, 11.7)
- moved R1 0.50 mm to (39.0, 18.2)
- moved R2 0.50 mm to (39.0, 23.0)
- moved R3 0.50 mm to (39.2, 27.8)
- moved R4 0.50 mm to (39.2, 32.5)
- moved R5 0.50 mm to (39.0, 8.75)
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Connections:
- new net +VIN1: C4.+, D1.C, IC1.2, R13.2, U$2.P$1, U$2.P$3, U$2.P$5
- new net BLU_PWM2: JP2.1, R12.2
- new net GRN_PWM2: JP2.2, R8.2
- new net N$1: Q7.D, U$2.P$4
- new net N$11: C3.1, CN2.PWR, IC1.3
- new net N$12: C5.+, D1.A, IC1.1, R13.1, R14.2
- new net N$2: Q10.1, Q7.G, R8.1
- new net N$3: Q11.1, Q8.G, R10.1
- new net N$4: Q12.1, Q9.G, R12.1
- new net N$5: Q10.2, Q7.S, R7.2
- new net N$6: Q11.2, Q8.S, R9.2
- new net N$7: Q12.2, Q9.S, R11.2
- new net N$8: Q8.D, U$2.P$2
- new net N$9: Q9.D, U$2.P$6
- new net RED_PWM2: JP2.3, R10.2
- net GND: now also C3.2, C4.-, C5.-, CN2.GND, CN2.GNDBREAK, Q10.3, Q11.3, Q12.3, R11.1, R14.1, R7.1, R9.1
Routing:
- net +VIN1: track 0.00 -> 76.9 mm
- net RED_PWM2: track 0.00 -> 50.5 mm
- net N$4: track 0.00 -> 47.4 mm
- net N$3: track 0.00 -> 47.2 mm
- net N$2: track 0.00 -> 47.2 mm
- net GRN_PWM2: track 0.00 -> 45.3 mm
- net N$12: track 0.00 -> 32.5 mm
- net N$8: track 0.00 -> 32.2 mm
- net BLU_PWM2: track 0.00 -> 28.4 mm
- net N$34: track 0.00 -> 26.0 mm
- net N$33: track 0.00 -> 26.0 mm
- net N$32: track 0.00 -> 26.0 mm
- net N$31: track 0.00 -> 26.0 mm
- net N$16: track 0.00 -> 26.0 mm
- net N$15: track 0.00 -> 26.0 mm
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Other:
- board size 52.5 x 38 mm -> 80 x 79 mm
- board text added: "SJSU 2018"

Commit message: frankly, I've forgotten all the changes I've made but it's a lot
Parts:
- added +, -: WIREPAD3,81/1,4, wirepad:3,81/1,4
- added J1, J4: 2p-2.54, Seeed-Connector:H2-2.54
- added J2, J3: 1X2-3.5MM, adafruit:1X2-3.5MM
- added LED1: (no value), led:LED3MM
- added R15: (no value), resistor:0207/12
- D1: value 1N4004 -> 1N4002
- R1, R3, R5: value (none) -> 100K
- moved CN1 1.00 mm to (-3.00, 28.5)
Connections:
- new net N$41: LED1.A, R15.2
- new net N$42: +.1, R15.1
- new net N$43: -.1, LED1.K
- net +VIN: now also J1.1, J2.1
- net GND: now also J1.2, J2.2, J3.2, J4.2
- net N$11: now also J3.1, J4.1
Routing:
- net N$42: track 0.00 -> 39.9 mm
- net N$43: track 0.00 -> 27.0 mm
- net N$34: track 26.0 -> 0.00 mm
- net N$33: track 26.0 -> 0.00 mm
- net N$32: track 26.0 -> 0.00 mm
- net N$31: track 26.0 -> 0.00 mm
- net N$16: track 26.0 -> 0.00 mm
- net N$15: track 26.0 -> 0.00 mm
- net N$14: track 26.0 -> 0.00 mm
- net N$13: track 26.0 -> 0.00 mm
- net N$41: track 0.00 -> 22.7 mm
- net N$35: track 21.9 -> 0.00 mm
- net N$23: track 21.9 -> 0.00 mm
- net N$37: track 15.9 -> 0.00 mm
- net N$25: track 15.9 -> 0.00 mm
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Other:
- board size 80 x 79 mm -> 80 x 79.3 mm
- board text added: "+"
- board text added: "-"
