File: lumiled_driver.sch (EAGLE design)
At the start: 17 parts, among them Q1 IRF520, Q2 2N3904, Q3 IRF520, Q4 2N3904, Q5 IRF520, Q6 2N3904

Commit message: just a commit
Parts:
- U$1: value LUMILED_5LED -> LUMILED_PARALLEL; device lumiled_led:LUMILED_5LED -> lumiled_led:LUMILED_PARALLEL
Changed lines of the file:
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@@
 </classes>
 <parts>
-<part name="U$1" library="lumiled_led" deviceset="LUMILED_5LED" device=""/>
 <part name="GND5" library="supply1" library_urn="urn:adsk.eagle:library:371" deviceset="GND" device=""/>
 <part name="C1" library="rcl" library_urn="urn:adsk.eagle:library:334" deviceset="C-US" device="025-024X044" package3d_urn="urn:adsk.eagle:package:23630/1" value="100nF"/>
@@
 <part name="JP1" library="pinhead" library_urn="urn:adsk.eagle:library:325" deviceset="PINHD-1X3" device="" package3d_urn="urn:adsk.eagle:package:22458/2"/>
 <part name="C2" library="resistor" library_urn="urn:adsk.eagle:library:348" deviceset="CPOL-US" device="TT2D5" package3d_urn="urn:adsk.eagle:package:25805/1" value="1uF"/>
+<part name="U$1" library="lumiled_led" deviceset="LUMILED_PARALLEL" device=""/>
 </parts>
 <sheets>
@@
 </plain>
 <instances>
-<instance part="U$1" gate="G$1" x="83.82" y="12.7"/>
 <instance part="GND5" gate="1" x="35.56" y="2.54"/>
 <instance part="C1" gate="G$1" x="27.94" y="20.32" rot="R180"/>
@@
 <instance part="JP1" gate="A" x="17.78" y="-33.02" rot="R180"/>
 <instance part="C2" gate="G$1" x="35.56" y="20.32" rot="R180"/>
+<instance part="U$1" gate="G$1" x="83.82" y="12.7"/>
 </instances>
 <busses>
@@
 <junction x="27.94" y="15.24"/>
 <wire x1="35.56" y1="17.78" x2="35.56" y2="15.24" width="0.1524" layer="91"/>
-<pinref part="U$1" gate="G$1" pin="RED+"/>
 <wire x1="55.88" y1="15.24" x2="45.72" y2="15.24" width="0.1524" layer="91"/>
 <junction x="45.72" y="15.24"/>
 <wire x1="35.56" y1="15.24" x2="45.72" y2="15.24" width="0.1524" layer="91"/>
 <junction x="35.56" y="15.24"/>
-<pinref part="U$1" gate="G$1" pin="GRN+"/>
 <wire x1="55.88" y1="17.78" x2="45.72" y2="17.78" width="0.1524" layer="91"/>
 <junction x="45.72" y="17.78"/>
 <wire x1="45.72" y1="15.24" x2="45.72" y2="17.78" width="0.1524" layer="91"/>
-<pinref part="U$1" gate="G$1" pin="BLU+"/>
 <wire x1="55.88" y1="12.7" x2="45.72" y2="12.7" width="0.1524" layer="91"/>
 <junction x="45.72" y="12.7"/>
@@
 <wire x1="22.86" y1="15.24" x2="27.94" y2="15.24" width="0.1524" layer="91"/>
 <pinref part="C2" gate="G$1" pin="+"/>
+<pinref part="U$1" gate="G$1" pin="GRN+"/>
+<pinref part="U$1" gate="G$1" pin="RED+"/>
+<pinref part="U$1" gate="G$1" pin="BLU+"/>
 </segment>
 </net>
 <net name="N$10" class="0">
 <segment>
-<pinref part="U$1" gate="G$1" pin="GRN-"/>
 <wire x1="73.66" y1="0" x2="73.66" y2="-10.16" width="0.1524" layer="91"/>
 <pinref part="Q1" gate="G$1" pin="D"/>
+<pinref part="U$1" gate="G$1" pin="GRN-"/>
 </segment>
 </net>
@@
 <net name="N$26" class="0">
 <segment>
-<pinref part="U$1" gate="G$1" pin="RED-"/>
 <wire x1="81.28" y1="0" x2="86.36" y2="0" width="0.1524" layer="91"/>
 <wire x1="86.36" y1="0" x2="86.36" y2="-10.16" width="0.1524" layer="91"/>
 <pinref part="Q3" gate="G$1" pin="D"/>
 <wire x1="86.36" y1="-10.16" x2="91.44" y2="-10.16" width="0.1524" layer="91"/>
+<pinref part="U$1" gate="G$1" pin="RED-"/>
 </segment>
 </net>
 <net name="N$27" class="0">
 <segment>
-<pinref part="U$1" gate="G$1" pin="BLU-"/>
 <wire x1="88.9" y1="0" x2="104.14" y2="0" width="0.1524" layer="91"/>
 <wire x1="104.14" y1="0" x2="104.14" y2="-10.16" width="0.1524" layer="91"/>
 <pinref part="Q5" gate="G$1" pin="D"/>
 <wire x1="104.14" y1="-10.16" x2="109.22" y2="-10.16" width="0.1524" layer="91"/>
-</segment>
-</net>
+<pinref part="U$1" gate="G$1" pin="BLU-"/>
+</segment>
+</net>

Commit message: -wow it's been a while since the last commit
Parts:
- R1, R2, R3, R4, R5, R6: device rcl:R-US_0204/7 -> resistor:R-US_0411/12
Changed lines of the file:
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@@
 <?xml version="1.0" encoding="utf-8"?>
 <!DOCTYPE eagle SYSTEM "eagle.dtd">
-<eagle version="8.3.1">
+<eagle version="8.4.1">
 <drawing>
 <settings>
@@
 <part name="Q4" library="transistor-npn" deviceset="2N3904" device=""/>
 <part name="Q6" library="transistor-npn" deviceset="2N3904" device=""/>
-<part name="R2" library="rcl" deviceset="R-US_" device="0204/7"/>
-<part name="R1" library="rcl" deviceset="R-US_" device="0204/7"/>
+<part name="R2" library="resistor" library_urn="urn:adsk.eagle:library:348" deviceset="R-US_" device="0411/12" package3d_urn="urn:adsk.eagle:package:26091/1"/>
+<part name="R1" library="resistor" library_urn="urn:adsk.eagle:library:348" deviceset="R-US_" device="0411/12" package3d_urn="urn:adsk.eagle:package:26091/1"/>
 <part name="GND2" library="supply1" library_urn="urn:adsk.eagle:library:371" deviceset="GND" device=""/>
-<part name="R4" library="rcl" deviceset="R-US_" device="0204/7"/>
-<part name="R3" library="rcl" deviceset="R-US_" device="0204/7"/>
-<part name="R6" library="rcl" deviceset="R-US_" device="0204/7"/>
-<part name="R5" library="rcl" deviceset="R-US_" device="0204/7"/>
+<part name="R4" library="resistor" library_urn="urn:adsk.eagle:library:348" deviceset="R-US_" device="0411/12" package3d_urn="urn:adsk.eagle:package:26091/1"/>
+<part name="R3" library="resistor" library_urn="urn:adsk.eagle:library:348" deviceset="R-US_" device="0411/12" package3d_urn="urn:adsk.eagle:package:26091/1"/>
+<part name="R6" library="resistor" library_urn="urn:adsk.eagle:library:348" deviceset="R-US_" device="0411/12" package3d_urn="urn:adsk.eagle:package:26091/1"/>
+<part name="R5" library="resistor" library_urn="urn:adsk.eagle:library:348" deviceset="R-US_" device="0411/12" package3d_urn="urn:adsk.eagle:package:26091/1"/>
 <part name="CN1" library="adafruit" deviceset="DCBARREL" device="PTH"/>
 <part name="JP1" library="pinhead" library_urn="urn:adsk.eagle:library:325" deviceset="PINHD-1X3" device="" package3d_urn="urn:adsk.eagle:package:22458/2"/>

Commit message: -sent out to elecrow for fabrication
Parts:
- added C3: 100nF, rcl:C-US025-024X044
- added C4: 1uF, resistor:CPOL-USTT2D5
- added C5: 10uF, resistor:CPOL-USTT2D5
- added CN2: (no value), adafruit:DCBARRELPTH
- added D1: 1N4004, diode:1N4004
- added IC1: (no value), v-reg:LM317TL
- added JP2: (no value), pinhead:PINHD-1X3
- added Q10, Q11, Q12: 2N3904, transistor-npn:2N3904
- added Q7, Q8, Q9: IRF520, transistor-power:IRF520
- added R10, R11, R12, R13, R14, R7, R8, R9: (no value), resistor:R-US_0411/12
- added U$2: LUMILED_PARALLEL, lumiled_led:LUMILED_PARALLEL
Connections:
- new net +VIN1: C4.+, D1.C, IC1.OUT, R13.2, U$2.BLU+, U$2.GRN+, U$2.RED+
- new net BLU_PWM2: JP2.1, R12.2
- new net GRN_PWM2: JP2.2, R8.2
- new net N$1: Q7.D, U$2.GRN-
- new net N$11: C3.1, CN2.PWR, IC1.IN
- new net N$12: C5.+, D1.A, IC1.ADJ, R13.1, R14.2
- new net N$2: Q10.C, Q7.G, R8.1
- new net N$3: Q11.C, Q8.G, R10.1
- new net N$4: Q12.C, Q9.G, R12.1
- new net N$5: Q10.B, Q7.S, R7.2
- new net N$6: Q11.B, Q8.S, R9.2
- new net N$7: Q12.B, Q9.S, R11.2
- new net N$8: Q8.D, U$2.RED-
- new net N$9: Q9.D, U$2.BLU-
- new net RED_PWM2: JP2.3, R10.2
- net GND: now also C3.2, C4.-, C5.-, CN2.GND, CN2.GNDBREAK, Q10.E, Q11.E, Q12.E, R11.1, R14.1, R7.1, R9.1
Other:
- moved on the sheet: C1, C2, CN1, JP1, Q1, Q2, Q3, Q4, Q5, Q6, R1, R2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

Commit message: frankly, I've forgotten all the changes I've made but it's a lot
Parts:
- added +, -: WIREPAD3,81/1,4, wirepad:WIREPAD3,81/1,4
- added J1, J4: 2p-2.54, Seeed-Connector:DIP-BLACK-MALE-HEADER-VERT(2P-2.54)
- added J2, J3: 1X2-3.5MM, adafruit:1X2-3.5MM
- added LED1: (no value), led:LED3MM
- added R15: (no value), resistor:R-US_0207/12
- D1: value 1N4004 -> 1N4002
- R1, R3, R5: value (none) -> 100K
Connections:
- new net N$41: LED1.A, R15.2
- new net N$42: +.P, R15.1
- new net N$43: -.P, LED1.C
- net +VIN: now also J1.1, J2.1
- net GND: now also J1.2, J2.2, J3.2, J4.2
- net N$11: now also J3.1, J4.1
Other:
- moved on the sheet: C1, C2, C3, C4, C5, CN1, CN2, D1, IC1, JP1, JP2, Q1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
