File: huzzah32_driver.sch (EAGLE design)
At the start: 9 parts, among them IC1 7805T, J1 1X2-3.5MM, X1 C-GRID-16-70543, X2 C-GRID-12-70543, X3 22-23-2021, X4 22-23-2021

Commit message: I've been working on this for like 6 hours and now it's 4am you expect me to write a commit message? -finished the board
Parts:
- added C3: 330nF, resistor:C-US050-035X075
- added C4: 100nF, resistor:C-US050-035X075
- added CN2: (no value), adafruit:DCBARRELPTH
- added IC2: 7805T, linear:7805T
- added J2, J3, J4: 1X2-3.5MM, adafruit:1X2-3.5MM
- added JP1, JP2: (no value), pinhead:PINHD-1X24
- added X10, X7, X8, X9: 22-23-2021, con-molex:22-23-2021
- added X5: C-GRID-16-70543, lumiled_boards:C-GRID-16-70543
- added X6: C-GRID-12-70543, lumiled_boards:C-GRID-12-70543
Connections:
- removed net A0_DAC2: X1-12.S
- removed net A1_DAC1: X1-11.S
- removed net A2_I34: X1-10.S
- removed net A3_I39: X1-9.S
- removed net A4_IO36: X1-8.S
- removed net A5_IO4: X1-7.S
- removed net EN: X2-2.S
- removed net IO12_A11: X2-5.S
- removed net IO13_A12: X2-4.S
- removed net IO14_A6: X2-10.S
- removed net IO15_A8: X2-8.S
- removed net IO16: X1-3.S
- removed net IO17: X1-2.S
- removed net IO21: X1-1.S
- removed net IO27_A10: X2-6.S
- removed net IO32_A7: X2-9.S
- removed net IO33_A9: X2-7.S
- removed net MISO: X1-4.S
- removed net MOSI: X1-5.S
- removed net N$26: X1-14.S
- removed net RESET: X1-16.S
- removed net SCK: X1-6.S
- removed net SCL: X2-11.S
- removed net SDA: X2-12.S
- removed net VBAT: X2-1.S
- new net A0_DAC2_B1: JP1.1, X1-12.S
- new net A0_DAC2_B2: JP2.1, X5-12.S
- new net A1_DAC1_B1: JP1.2, X1-11.S
- new net A1_DAC1_B2: JP2.2, X5-11.S
- new net A2_I34_B1: JP1.3, X1-10.S
- new net A2_I34_B2: JP2.3, X5-10.S
- new net A3_I39_B1: JP1.4, X1-9.S
- new net A3_I39_B2: JP2.4, X5-9.S
- new net A4_IO36_B1: JP1.5, X1-8.S
- new net A4_IO36_B2: JP2.5, X5-8.S
- new net A5_IO4_B1: JP1.6, X1-7.S
- new net A5_IO4_B2: JP2.6, X5-7.S
- new net IO12_A11_B1: JP1.12, X2-5.S
- new net IO12_A11_B2: JP2.12, X6-5.S
- new net IO13_A12_B1: JP1.13, X2-4.S
- new net IO13_A12_B2: JP2.13, X6-4.S
- new net IO14_A6_B1: JP1.7, X2-10.S
- new net IO14_A6_B2: JP2.7, X6-10.S
- new net IO15_A8_B1: JP1.9, X2-8.S
- new net IO15_A8_B2: JP2.9, X6-8.S
- new net IO16_B1: JP1.14, X1-3.S
- new net IO16_B2: JP2.14, X5-3.S
- new net IO17_B1: JP1.15, X1-2.S
- new net IO17_B2: JP2.15, X5-2.S
- new net IO21_B1: JP1.16, X1-1.S
- new net IO21_B2: JP2.16, X5-1.S
- new net IO27_A10_B1: JP1.11, X2-6.S
- new net IO27_A10_B2: JP2.11, X6-6.S
- new net IO32_A7_B1: JP1.8, X2-9.S
- new net IO32_A7_B2: JP2.8, X6-9.S
- new net IO33_A9_B1: JP1.10, X2-7.S
- new net IO33_A9_B2: JP2.10, X6-7.S
- new net MISO_B1: JP1.20, X1-4.S
- new net MISO_B2: JP2.20, X5-4.S
- new net MOSI_B1: JP1.19, X1-5.S
- new net MOSI_B2: JP2.19, X5-5.S
- new net SCK_B1: JP1.21, X1-6.S
- new net SCK_B2: JP2.21, X5-6.S
- new net SCL_B1: JP1.17, X2-11.S
- new net SCL_B2: JP2.17, X6-11.S
- new net SDA_B1: JP1.18, X2-12.S
- new net SDA_B2: JP2.18, X6-12.S
- net +3V3: now also X10-2.S, X5-15.S, X9-2.S
- net +5V: now also C4.1, IC2.VO, X6-3.S, X8-2.S
- net GND: now also C3.2, C4.2, CN2.GND, CN2.GNDBREAK, IC2.GND, J2.1, J3.1, J4.1, JP1.22, JP1.23, JP1.24, JP2.22, JP2.23, JP2.24, X10-1.S, X5-13.S, X7-1.S, X8-1.S, X9-1.S
- net V+: now also C3.1, CN2.PWR, IC2.VI, J2.2, J3.2, J4.2, X7-2.S
Other:
- note added: "Board 1"
- note added: "Board 2"
- moved on the sheet: X1-1, X1-10, X1-11, X1-12, X1-13, X1-14, X1-15, X1-16, X1-2, X1-3, X1-4, X1-5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
